File: HW2/New_Project/HW2.sch (EAGLE design)
At the start: 22 parts, among them J3 USB-MB-H

Commit message: added board
Parts:
- renumbered U$2 to VOLTAGEMAKER
Connections:
- removed net N$1: C2.1, C4.+, U$7.2, VOLTAGEMAKER.2.VOUT
- new net N$2: J3.VBUS, U$7.2
- net +3V3: now also C2.1, C4.+, VOLTAGEMAKER.2.VOUT; no longer U$7.1
- net +5V: now also U$7.3; no longer J3.VBUS
Other:
- moved on the sheet: U$7
Changed lines of the file:
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@@
 <part name="LED1" library="HW2" deviceset="LED" device="3MM" value="RED"/>
 <part name="LED2" library="HW2" deviceset="LED" device="3MM" value="GREEN"/>
-<part name="U$2" library="HW2" deviceset="MCP1702" device=""/>
+<part name="VOLTAGEMAKER" library="HW2" deviceset="MCP1702" device=""/>
 <part name="U$3" library="HW2" deviceset="OSC" device=""/>
 <part name="U$6" library="HW2" deviceset="PICKIT" device=""/>
@@
 <part name="USRPB" library="HW2" deviceset="PB" device=""/>
 <part name="MCLRPB" library="HW2" deviceset="PB" device=""/>
-<part name="+3V1" library="HW2" deviceset="+3V3" device=""/>
 <part name="+3V2" library="HW2" deviceset="+3V3" device=""/>
 <part name="GND1" library="HW2" deviceset="GND" device=""/>
@@
 <part name="+3V10" library="HW2" deviceset="+3V3" device=""/>
 <part name="GND12" library="HW2" deviceset="GND" device=""/>
+<part name="+3V1" library="HW2" deviceset="+3V3" device=""/>
 </parts>
 <sheets>
@@
 <instance part="LED1" gate="G$1" x="50.8" y="33.02" rot="R90"/>
 <instance part="LED2" gate="G$1" x="50.8" y="20.32" rot="R90"/>
-<instance part="U$2" gate="G$1" x="-2.54" y="63.5"/>
+<instance part="VOLTAGEMAKER" gate="G$1" x="-2.54" y="63.5"/>
 <instance part="U$3" gate="G$1" x="55.88" y="0"/>
 <instance part="U$6" gate="G$1" x="-68.58" y="-2.54"/>
@@
 <instance part="R3" gate="G$1" x="-50.8" y="35.56" rot="R90"/>
 <instance part="R4" gate="G$1" x="-50.8" y="15.24" rot="R90"/>
-<instance part="U$7" gate="G$1" x="48.26" y="55.88" rot="R180"/>
+<instance part="U$7" gate="G$1" x="-40.64" y="76.2"/>
 <instance part="J3" gate="G$1" x="-60.96" y="66.04" rot="R180"/>
 <instance part="USRPB" gate="G$1" x="-66.04" y="10.16"/>
 <instance part="MCLRPB" gate="G$1" x="-66.04" y="30.48"/>
-<instance part="+3V1" gate="G$1" x="53.34" y="68.58"/>
 <instance part="+3V2" gate="G$1" x="-88.9" y="50.8"/>
 <instance part="GND1" gate="1" x="68.58" y="-38.1" rot="R90"/>
@@
 <instance part="+3V10" gate="G$1" x="-58.42" y="-35.56" rot="R270"/>
 <instance part="GND12" gate="1" x="-55.88" y="-38.1" rot="R90"/>
+<instance part="+3V1" gate="G$1" x="35.56" y="63.5" rot="R270"/>
 </instances>
 <busses>
 </busses>
 <nets>
-<net name="N$1" class="0">
-<segment>
-<pinref part="U$2" gate="G$1" pin="2.VOUT"/>
-<pinref part="C4" gate="G$1" pin="+"/>
-<wire x1="27.94" y1="63.5" x2="17.78" y2="63.5" width="0.1524" layer="91"/>
-<pinref part="C2" gate="G$1" pin="1"/>
-<junction x="17.78" y="63.5"/>
-<wire x1="17.78" y1="63.5" x2="15.24" y2="63.5" width="0.1524" layer="91"/>
-<wire x1="27.94" y1="63.5" x2="48.26" y2="63.5" width="0.1524" layer="91"/>
-<junction x="27.94" y="63.5"/>
-<pinref part="U$7" gate="G$1" pin="2"/>
-<wire x1="48.26" y1="63.5" x2="48.26" y2="60.96" width="0.1524" layer="91"/>
-</segment>
-</net>
 <net name="N$6" class="0">
 <segment>
@@
 </net>
 <net name="+3V3" class="0">
-<segment>
-<pinref part="U$7" gate="G$1" pin="1"/>
-<pinref part="+3V1" gate="G$1" pin="+3V3"/>
-<wire x1="53.34" y1="66.04" x2="53.34" y2="60.96" width="0.1524" layer="91"/>
-</segment>
 <segment>
 <pinref part="C5" gate="G$1" pin="1"/>
@@
 <pinref part="+3V10" gate="G$1" pin="+3V3"/>
 </segment>
+<segment>
+<pinref part="VOLTAGEMAKER" gate="G$1" pin="2.VOUT"/>
+<pinref part="C4" gate="G$1" pin="+"/>
+<wire x1="27.94" y1="63.5" x2="17.78" y2="63.5" width="0.1524" layer="91"/>
+<pinref part="C2" gate="G$1" pin="1"/>
+<junction x="17.78" y="63.5"/>
+<wire x1="17.78" y1="63.5" x2="15.24" y2="63.5" width="0.1524" layer="91"/>
+<wire x1="27.94" y1="63.5" x2="33.02" y2="63.5" width="0.1524" layer="91"/>
+<pinref part="+3V1" gate="G$1" pin="+3V3"/>
+</segment>
 </net>
 <net name="GND" class="0">
 <segment>
-<pinref part="U$2" gate="G$1" pin="1.GND"/>
+<pinref part="VOLTAGEMAKER" gate="G$1" pin="1.GND"/>
 <pinref part="C2" gate="G$1" pin="2"/>
 <wire x1="-2.54" y1="53.34" x2="17.78" y2="53.34" width="0.1524" layer="91"/>
@@
 <wire x1="-25.4" y1="53.34" x2="-2.54" y2="53.34" width="0.1524" layer="91"/>
 <pinref part="J3" gate="G$1" pin="GND"/>
-<wire x1="-58.42" y1="66.04" x2="-30.48" y2="66.04" width="0.1524" layer="91"/>
-<wire x1="-30.48" y1="66.04" x2="-30.48" y2="53.34" width="0.1524" layer="91"/>
-<wire x1="-30.48" y1="53.34" x2="-25.4" y2="53.34" width="0.1524" layer="91"/>
+<wire x1="-58.42" y1="66.04" x2="-33.02" y2="66.04" width="0.1524" layer="91"/>
+<wire x1="-33.02" y1="66.04" x2="-33.02" y2="53.34" width="0.1524" layer="91"/>
+<wire x1="-33.02" y1="53.34" x2="-25.4" y2="53.34" width="0.1524" layer="91"/>
 <junction x="-25.4" y="53.34"/>
 <pinref part="GND2" gate="1" pin="GND"/>
@@
 <net name="+5V" class="0">
 <segment>
-<pinref part="U$2" gate="G$1" pin="2.VIN"/>
+<pinref part="VOLTAGEMAKER" gate="G$1" pin="2.VIN"/>
 <pinref part="C1" gate="G$1" pin="1"/>
 <wire x1="-25.4" y1="63.5" x2="-20.32" y2="63.5" width="0.1524" layer="91"/>
-<pinref part="J3" gate="G$1" pin="VBUS"/>
-<wire x1="-58.42" y1="63.5" x2="-25.4" y2="63.5" width="0.1524" layer="91"/>
 <junction x="-25.4" y="63.5"/>
 <pinref part="P+1" gate="1" pin="+5V"/>
+<pinref part="U$7" gate="G$1" pin="3"/>
+<wire x1="-35.56" y1="71.12" x2="-27.94" y2="71.12" width="0.1524" layer="91"/>
+<wire x1="-27.94" y1="71.12" x2="-27.94" y2="63.5" width="0.1524" layer="91"/>
+<wire x1="-27.94" y1="63.5" x2="-25.4" y2="63.5" width="0.1524" layer="91"/>
 </segment>
 <segment>
@@
 </segment>
 </net>
+<net name="N$2" class="0">
+<segment>
+<pinref part="U$7" gate="G$1" pin="2"/>
+<wire x1="-40.64" y1="71.12" x2="-40.64" y2="63.5" width="0.1524" layer="91"/>
+<pinref part="J3" gate="G$1" pin="VBUS"/>
+<wire x1="-40.64" y1="63.5" x2="-58.42" y2="63.5" width="0.1524" layer="91"/>
+</segment>
+</net>
